Commit message: Add draft of model changes

File: model/urdf/arm.urdf (robot description, URDF)
Before this commit: robot Workshop Arm, 3 links, 2 joints
Links:
- removed link link1
- removed link link2
- added link link0; visual mesh filename=package://model/meshes/link0.stl scale=0.001 0.001 0.001
- link base_link: geometry visual mesh filename=package://model/meshes/base_link.stl scale=0.001 0.001 0.001
Joints:
- removed joint base_link_to_link1
- removed joint link1_to_link2
- added joint base_link_to_link0: type fixed, parent base_link, child link0, origin xyz=0 0 0
